File: dac-controller/board.sch (EAGLE design)
At the start: 39 parts, among them IC1 LM317MABT, IC2 ISO7220C, IC3 74HCT595D

Commit message: added dc-ac convert, added correct connector(s) for VFD, ripped up some traces to move things around
Parts:
- removed VFL: (no value), con-lstb:MA10-2
- added C10, C9: 0.1uF, rcl:C-EUC1206
- added C11: 0.01uF, rcl:C-EUC1206
- added C12: 2700uF, rcl:CPOL-EUE3.5-8
- added CON1-10, CON11-20, CON21-30: (no value), con-lsta:FE10-1
- added IC4: NE555, st-microelectronics:NE555
- added L1: (no value), rcl:L-EU0204/5
- added R1: 100R, rcl:R-EU_0207/10
- added R3: 10k, rcl:R-EU_R1206
- added R5: 125k, rcl:R-EU_R1206
- added R6: 100, rcl:R-EU_R1206
- added T1: (no value), transistor:-NPN-TO92
- added T2: (no value), transistor:-PNP-TO92
- added U$5: TRAFO-1:1, archi_laptop:TRAFO-1:1
- IC1: value LM317MABT -> (none); device v-reg:LM317MABT -> v-reg:LM317TS
Connections:
- new net N$11: CON11-20.7, U$4.OUT5
- new net N$12: CON21-30.10, U$4.OUT17
- new net N$13: CON21-30.9, U$4.OUT16
- new net N$49: R6.1, T1.B, T2.B
- new net N$54: C12.-, L1.2
- new net N$7: CON1-10.2, R1.2
- new net N$8: CON11-20.1, U$5.P$1
- new net N$9: CON11-20.2, U$5.P$2
- net 5V_RAW: now also C10.1, IC4./RES, IC4.VCC+, R1.1, R3.2, T1.C
- net GND: now also C10.2, C11.2, C9.2, CON1-10.1, CON21-30.6, IC4.GND, T2.C, U$5.P$3
- net N$19: now also CON21-30.8, U$4.OUT15; no longer U$4.OUT0, VFL.1
- net N$20: now also CON21-30.7, U$4.OUT14; no longer U$4.OUT1, VFL.2
- net N$21: now also CON21-30.5, U$4.OUT13; no longer U$4.OUT2, VFL.3
- net N$22: now also CON21-30.4, U$4.OUT12; no longer U$4.OUT3, VFL.4
- net N$23: now also CON21-30.3, U$4.OUT11; no longer U$4.OUT4, VFL.5
- net N$31: now also CON21-30.2, U$4.OUT10; no longer U$4.OUT6, VFL.7
- net N$32: now also CON21-30.1, U$4.OUT9; no longer U$4.OUT8, VFL.9
- net N$33: now also CON11-20.10, U$4.OUT8; no longer U$4.OUT10, VFL.11
- net N$34: now also CON11-20.9, U$4.OUT7; no longer U$4.OUT12, VFL.13
- net N$35: now also CON11-20.8, U$4.OUT6; no longer U$4.OUT14, VFL.15
- net N$36: now also CON11-20.6, U$4.OUT4; no longer U$4.OUT16, VFL.17
- net N$37: now also CON11-20.5, U$4.OUT3; no longer U$4.OUT18, VFL.19
- net N$38: now also CON11-20.4, U$4.OUT2; no longer U$4.OUT5, VFL.6
- net N$39: now also CON11-20.3, U$4.OUT1; no longer U$4.OUT7, VFL.8
- net N$40: now also C11.1, IC4.CON; no longer U$4.OUT9, VFL.10
- net N$41: now also IC4.DIS, R3.1, R5.2; no longer U$4.OUT11, VFL.12
- net N$42: now also C9.1, IC4.TRE, IC4.TRI, R5.1; no longer U$4.OUT13, VFL.14
- net N$43: now also IC4.OUT, R6.2; no longer U$4.OUT15, VFL.16
- net N$44: now also C12.+, T1.E, T2.E; no longer U$4.OUT17, VFL.18
- net N$45: now also L1.1, U$5.P$4; no longer U$4.OUT19, VFL.20
