File: car/v2/v1.brd (EAGLE design)
At the start: 50 x 50 mm, 18 parts, among them IC1 4066N, T1 2N3704

Commit message: updated board
Parts:
- moved 12V 0.79 mm to (3.17, 32.2)
- moved T1 0.32 mm to (9.68, 41.9)
Routing:
- net GND: track 9.05 -> 0.00 mm
- net N$1: track 48.8 -> 51.7 mm
- net DATA: track 34.3 -> 35.8 mm
- net N$4: track 42.5 -> 41.5 mm
- net CLK: track 37.3 -> 36.3 mm
- net N$18: track 45.4 -> 46.3 mm
- net 12V: track 7.88 -> 7.09 mm
- net V_RUN: track 7.64 -> 8.15 mm
Other:
- board text added: "Software: https://github.com/visualapproach/Volvo-melbus PCB: https://github.com/archi/boards Batch 2, Rev 2"
- board text added: "Solder IC1 first (other side)"
- board text removed: "Software: https://github.com/visualapproach/Volvo-melbus PCB: https://github.com/archi/boards Batch 1"
- board text removed: "Solder IC1 first!"
